File: sch_pcb/PiPtr.kicad_pcb (KiCad board)
At the start: 4 copper layers, 105 x 141.9 mm, 358 parts, among them J101 GLOBAL_LINK_LEFT, J102 GLOBAL_LINK_RIGHT, J107 RASPBERRY_PI, J111 FP_PIXEL, J112 AM2302, J113 I2C1_5V, J114 I2C0_3v3, J117 OLED_SSD1306, J201 TO_SOUNDCARD, J202 FROM_SOUNDCARD, J203 Radio Port, J204 DB9_FEMALE, J301 SPARE, J302 SPARE, J303 SPARE, J304 SPARE, J305 USER_GPIO_2, J306 SPARE, J307 SPARE, J308 USER_GPIO_1, J309 SPARE, J310 SPARE, J311 USER_ADC, J313 SPARE, J314 SPARE, J315 12VDC_IN, J401 TO_SOUNDCARD, J402 FROM_SOUNDCARD, J403 Radio Port, J404 DB9_FEMALE, Q101 2N7000, Q102 2N7000, Q103 2N7000, Q104 2N7000, Q105 2N7000, Q201 2N7000, Q202 2N7000, Q203 2N7000, Q301 SPARE, Q302 SPARE, Q401 2N7000, Q402 2N7000, Q403 2N7000, U101 MCP23017, U102 IP4234CZ6, U103 MCP4351, U104 74HCT138, U105 74LV1T125, U106 MCP4351, U107 MCP4351, U108 IP4234CZ6, U109 IP4234CZ6, U110 74LV1T125, U111 74LV1T125, U112 74LV1T125, U113 74LV1T125, U201 MCP6004N, U202 74LVC1G3157, U203 74LVC1G3157, U204 74LVC4066, U205 MCP6004N, U206 74LVC1G3157, U207 MCP6S26, U301 MCP23017, U302 SPARE, U303 SPARE, U304 MCP3008, U305 MCP1703A-2502/MB, U306 TPS54302, U401 MCP6004N, U402 74LVC1G3157, U403 74LVC1G3157, U404 74LVC4066, U405 MCP6004N, U406 74LVC1G3157, U407 MCP6S26, U501 CM108B, U502 CM108B, U503 TUSB2036, Y501 6MHz

Commit message: Update from latest round of emails
Change connectors - use correct footprint for DE9F.  Add chassis connector as DE9M, AUX_IO connectors as 116-pin ribbon, expected to transition to DA15 with a cable.  
Remove screw terminals for 12V input as it now comes in on chassis connector
Remove third EEPOT package
Move stuff off PCB in preparation to incorporate all the schematic updates.
Parts:
- removed C202, C402: 10u, lib:smd0603
- removed C216, C416: 10u, lib:smd0805
- removed J201, J401: TO_SOUNDCARD, lib:TRS3.5_5
- removed J202, J402: FROM_SOUNDCARD, lib:TRS3.5_5
- removed J203, J403: Radio Port, lib:RibbonHeader2x5
- removed J311: USER_ADC, lib:RibbonHeader2x7
- removed J315: 12VDC_IN, ardai:Phoenix_2pin_3.5mm_conn_1984963
- removed R227, R427: 100k, lib:smd0603
- removed RJ45_8 (x2): VAL**, connect:RJ45_8
- removed TP301, TP302, TP303, TP304, TP305, TP306: TESTPOINT, lib:Wire_28AWG
- removed U106: MCP4351, lib:SSOP-20
- added C527: 10u, lib:smd0603, F.Cu at (369.2, 20.5)
- added C528: 10u, lib:smd0603, F.Cu at (369.2, 22.8)
- added P301: Chassis, lib:DE9M_Right_Angle, F.Cu at (108.0, 40.6)
- added R329, R330, R331: 33, lib:smd0603, F.Cu at (108.0, 179.7)
- added R515: 33R, lib:smd0603, F.Cu at (372.0, 20.5)
- added R516: 33R, lib:smd0603, F.Cu at (372.0, 22.8)
- added TP501: CH1_RIGHT, lib:Wire_28AWG, F.Cu at (389.9, 22.9)
- added TP502: CH2_RIGHT, lib:Wire_28AWG, F.Cu at (389.9, 30.0)
- added U307: IP4234CZ6, lib:SOT23-6, F.Cu at (108.0, 179.7)
- J204, J404: value DB9_FEMALE -> DE9F; footprint lib:DB9FC -> lib:DE9F_Right_Angle
- J305: value USER_GPIO_2 -> AUX_IO_1
- J308: value USER_GPIO_1 -> AUX_IO_2
- Q101, Q102, Q103, Q104, Q105: value 2N7000 -> BSS138
- moved TP106 302.6 mm to (412.6, 54.6)
- moved U111 81.5 mm to (200.0, 134.7)
- moved U112 81.5 mm to (203.8, 134.7)
- moved C318 81.5 mm to (218.9, 95.2)
- moved R314 81.5 mm to (218.9, 92.2)
- moved R319 81.5 mm to (217.4, 95.2)
- moved R321 81.5 mm to (222.0, 92.2)
- moved R322 81.5 mm to (220.5, 95.2)
- moved R323 81.5 mm to (222.0, 95.2)
- moved U301 81.5 mm to (213.4, 105.9)
- moved C303 81.5 mm to (202.4, 92.5)
- moved C304 81.5 mm to (201.7, 97.8)
- moved C305 81.5 mm to (203.2, 97.8)
- moved C314 81.5 mm to (207.0, 95.2)
- moved C315 81.5 mm to (210.1, 95.2)
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Connections:
- C505 pad 1: +5V -> Net-(C505-Pad1)
- C506 pad 1: +5V -> Net-(C505-Pad1)
- C507 pad 1: +5V -> Net-(C507-Pad1)
- C508 pad 1: +5V -> Net-(C507-Pad1)
- C509 pad 1: /CH1/FROM_SOUNDCARD -> Net-(C509-Pad1)
- C510 pad 1: /CH2/FROM_SOUNDCARD -> Net-(C510-Pad1)
- J112 pad 3: Net-(J112-Pad3) -> (no net)
- J117 pad 3: /SCL0_33 -> /SCL1_33
- J117 pad 4: /SDA0_33 -> /SDA1_33
- J305 pad 10: GND -> /Spares, GPIO, and ADC/SDA0_OUT
- J305 pad 11: Net-(J305-Pad11) -> /Spares, GPIO, and ADC/SCL0_OUT
- J305 pad 13: Net-(J305-Pad13) -> /Spares, GPIO, and ADC/ADC2
- J305 pad 15: Net-(J305-Pad15) -> /Spares, GPIO, and ADC/ADC3
- J305 pad 16: GND -> (no net)
- J305 pad 2: GND -> /Spares, GPIO, and ADC/GPA0
- J305 pad 3: Net-(J305-Pad3) -> /Spares, GPIO, and ADC/GPA1
- J305 pad 4: GND -> /Spares, GPIO, and ADC/GPA2
- J305 pad 5: Net-(J305-Pad5) -> /Spares, GPIO, and ADC/GPA3
- J305 pad 6: GND -> /Spares, GPIO, and ADC/GPA4
- J305 pad 7: Net-(J305-Pad7) -> /Spares, GPIO, and ADC/GPA5
- J305 pad 8: GND -> /Spares, GPIO, and ADC/GPA6
- J305 pad 9: Net-(J305-Pad9) -> /Spares, GPIO, and ADC/GPA7
- J307 pad 1: Net-(J307-Pad1) -> (no net)
- J308 pad 10: GND -> /Spares, GPIO, and ADC/SDA0_OUT
- J308 pad 11: Net-(J308-Pad11) -> /Spares, GPIO, and ADC/SCL0_OUT
- J308 pad 13: Net-(J308-Pad13) -> /Spares, GPIO, and ADC/ADC4
- J308 pad 15: Net-(J308-Pad15) -> /Spares, GPIO, and ADC/ADC5
- J308 pad 16: GND -> (no net)
- J308 pad 2: GND -> /Spares, GPIO, and ADC/GPB0
- J308 pad 3: Net-(J308-Pad3) -> /Spares, GPIO, and ADC/GPB1
- J308 pad 4: GND -> /Spares, GPIO, and ADC/GPB2
- J308 pad 5: Net-(J308-Pad5) -> /Spares, GPIO, and ADC/GPB3
- J308 pad 6: GND -> /Spares, GPIO, and ADC/GPB4
- J308 pad 7: Net-(J308-Pad7) -> /Spares, GPIO, and ADC/GPB5
- J308 pad 8: GND -> /Spares, GPIO, and ADC/GPB6
- J308 pad 9: Net-(J308-Pad9) -> /Spares, GPIO, and ADC/GPB7
- MTG301 pad 1: Net-(MTG301-Pad1) -> (no net)
- MTG302 pad 1: Net-(MTG302-Pad1) -> (no net)
- MTG303 pad 1: Net-(MTG303-Pad1) -> (no net)
- MTG304 pad 1: Net-(MTG304-Pad1) -> (no net)
- R230 pad 1: /CH1/TONE_FROM_SOUNDCARD -> Net-(R230-Pad1)
- R430 pad 1: /CH2/TONE_FROM_SOUNDCARD -> Net-(R430-Pad1)
- R504 pad 2: Net-(R504-Pad2) -> (no net)
- R506 pad 2: Net-(R506-Pad2) -> (no net)
- U101 pad 19: Net-(U101-Pad19) -> (no net)
- U101 pad 20: Net-(U101-Pad20) -> (no net)
- U103 pad 19: Net-(U103-Pad19) -> Net-(R236-Pad2)
- U103 pad 20: /CH1/TONE_FROM_SOUNDCARD -> /CH1/TONE_FROM_PI
- U104 pad 13: /~R811CS -> (no net)
- U107 pad 19: Net-(U107-Pad19) -> Net-(R436-Pad2)
- U107 pad 20: /CH2/TONE_FROM_SOUNDCARD -> /CH2/TONE_FROM_PI
- U113 pad 2: Net-(U113-Pad2) -> /MOSI_33
- U205 pad 5: Net-(U103-Pad19) -> Net-(R230-Pad1)
- U207 pad 12: Net-(U207-Pad12) -> (no net)
- U207 pad 6: Net-(U207-Pad6) -> (no net)
- U207 pad 7: Net-(U207-Pad7) -> (no net)
- U301 pad 1: Net-(J305-Pad1) -> /Spares, GPIO, and ADC/GPB0
- U301 pad 2: Net-(J305-Pad3) -> /Spares, GPIO, and ADC/GPB1
- U301 pad 21: Net-(J308-Pad1) -> /Spares, GPIO, and ADC/GPA0
- U301 pad 22: Net-(J308-Pad3) -> /Spares, GPIO, and ADC/GPA1
- U301 pad 23: Net-(J308-Pad5) -> /Spares, GPIO, and ADC/GPA2
- U301 pad 24: Net-(J308-Pad7) -> /Spares, GPIO, and ADC/GPA3
- U301 pad 25: Net-(J308-Pad9) -> /Spares, GPIO, and ADC/GPA4
- U301 pad 26: Net-(J308-Pad11) -> /Spares, GPIO, and ADC/GPA5
- U301 pad 27: Net-(J308-Pad13) -> /Spares, GPIO, and ADC/GPA6
- U301 pad 28: Net-(J308-Pad15) -> /Spares, GPIO, and ADC/GPA7
- U301 pad 3: Net-(J305-Pad5) -> /Spares, GPIO, and ADC/GPB2
- U301 pad 4: Net-(J305-Pad7) -> /Spares, GPIO, and ADC/GPB3
- U301 pad 5: Net-(J305-Pad9) -> /Spares, GPIO, and ADC/GPB4
- U301 pad 6: Net-(J305-Pad11) -> /Spares, GPIO, and ADC/GPB5
- U301 pad 7: Net-(J305-Pad13) -> /Spares, GPIO, and ADC/GPB6
- U301 pad 8: Net-(J305-Pad15) -> /Spares, GPIO, and ADC/GPB7
- U405 pad 5: Net-(U107-Pad19) -> Net-(R430-Pad1)
- U407 pad 12: Net-(U407-Pad12) -> (no net)
- U407 pad 6: Net-(U407-Pad6) -> (no net)
- U407 pad 7: Net-(U407-Pad7) -> (no net)
- U501 pad 1: Net-(U501-Pad1) -> (no net)
- U501 pad 11: Net-(U501-Pad11) -> (no net)
- U501 pad 12: Net-(U501-Pad12) -> (no net)
- U501 pad 13: Net-(U501-Pad13) -> (no net)
- U501 pad 15: Net-(U501-Pad15) -> (no net)
- U501 pad 17: Net-(U501-Pad17) -> (no net)
- U501 pad 18: Net-(U501-Pad18) -> (no net)
- U501 pad 19: Net-(U501-Pad19) -> (no net)
- U501 pad 2: Net-(U501-Pad2) -> (no net)
- U501 pad 20: Net-(U501-Pad20) -> (no net)
- U501 pad 21: Net-(U501-Pad21) -> (no net)
- U501 pad 25: Net-(U501-Pad25) -> (no net)
- U501 pad 28: Net-(U501-Pad28) -> (no net)
- U501 pad 29: +5V -> Net-(C505-Pad1)
- U501 pad 3: Net-(U501-Pad3) -> (no net)
- U501 pad 31: Net-(U501-Pad31) -> (no net)
- U501 pad 34: +5V -> Net-(C505-Pad1)
- U501 pad 39: Net-(U501-Pad39) -> (no net)
- U501 pad 4: Net-(U501-Pad4) -> (no net)
- U501 pad 40: Net-(U501-Pad40) -> (no net)
- U501 pad 43: Net-(U501-Pad43) -> (no net)
- U501 pad 44: Net-(U501-Pad44) -> (no net)
- U501 pad 45: Net-(U501-Pad45) -> (no net)
- U501 pad 46: Net-(U501-Pad46) -> (no net)
- U501 pad 47: Net-(U501-Pad47) -> (no net)
- U501 pad 48: Net-(U501-Pad48) -> (no net)
- U501 pad 5: Net-(U501-Pad5) -> (no net)
- U501 pad 6: Net-(U501-Pad6) -> (no net)
- U502 pad 1: Net-(U502-Pad1) -> (no net)
- U502 pad 11: Net-(U502-Pad11) -> (no net)
- U502 pad 12: Net-(U502-Pad12) -> (no net)
- U502 pad 13: Net-(U502-Pad13) -> (no net)
- U502 pad 15: Net-(U502-Pad15) -> (no net)
- U502 pad 17: Net-(U502-Pad17) -> (no net)
- U502 pad 18: Net-(U502-Pad18) -> (no net)
- U502 pad 19: Net-(U502-Pad19) -> (no net)
- U502 pad 2: Net-(U502-Pad2) -> (no net)
- U502 pad 20: Net-(U502-Pad20) -> (no net)
- U502 pad 21: Net-(U502-Pad21) -> (no net)
- U502 pad 25: Net-(U502-Pad25) -> (no net)
- U502 pad 28: Net-(U502-Pad28) -> (no net)
- U502 pad 29: +5V -> Net-(C507-Pad1)
- U502 pad 3: Net-(U502-Pad3) -> (no net)
- U502 pad 31: Net-(U502-Pad31) -> (no net)
- U502 pad 34: +5V -> Net-(C507-Pad1)
- U502 pad 39: Net-(U502-Pad39) -> (no net)
- U502 pad 4: Net-(U502-Pad4) -> (no net)
- U502 pad 40: Net-(U502-Pad40) -> (no net)
- U502 pad 43: Net-(U502-Pad43) -> (no net)
- U502 pad 44: Net-(U502-Pad44) -> (no net)
- U502 pad 45: Net-(U502-Pad45) -> (no net)
- U502 pad 46: Net-(U502-Pad46) -> (no net)
- U502 pad 47: Net-(U502-Pad47) -> (no net)
- U502 pad 48: Net-(U502-Pad48) -> (no net)
- U502 pad 5: Net-(U502-Pad5) -> (no net)
- U502 pad 6: Net-(U502-Pad6) -> (no net)
- U503 pad 13: Net-(U503-Pad13) -> (no net)
- U503 pad 17: Net-(U503-Pad17) -> (no net)
- U503 pad 19: Net-(U503-Pad19) -> (no net)
- U503 pad 20: Net-(U503-Pad20) -> (no net)
- U503 pad 32: Net-(U503-Pad32) -> (no net)
- U503 pad 5: Net-(U503-Pad5) -> (no net)
- U503 pad 9: Net-(U503-Pad9) -> (no net)
Routing:
- net (no net): track 0.00 -> 256.8 mm, vias 0 -> 8
- net +5V: track 409.8 -> 272.9 mm, vias 25 -> 23
- net /PTT1D: track 100.6 -> 0.00 mm, vias 1 -> 0
- net /~CTCSS1: track 93.4 -> 0.00 mm, vias 1 -> 0
- net /COR1: track 85.1 -> 0.00 mm, vias 1 -> 0
- net /RX1_BUS2_EN: track 76.9 -> 0.00 mm, vias 1 -> 0
- net /RX1_BUS1_EN: track 69.8 -> 0.00 mm, vias 2 -> 0
- net /RX1_LOCAL_EN: track 68.2 -> 0.00 mm, vias 2 -> 0
- net /~R03CS: track 61.5 -> 0.00 mm, vias 4 -> 0
- net /PORT1_DET_EN: track 61.0 -> 0.00 mm, vias 2 -> 0
- net /RX1_BUS3_EN: track 69.7 -> 10.3 mm, vias 2 -> 1
- net /SDA1_5: track 99.7 -> 46.3 mm
- net SCLK_5: track 134.8 -> 82.1 mm, vias 6 -> 3
- net /~PGA1_CS: track 51.7 -> 0.00 mm, vias 4 -> 0
- net /RX2_BUS1_EN: track 56.5 -> 9.36 mm, vias 4 -> 1
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Other:
- board size 105 x 141.9 mm -> 101.6 x 141.7 mm

Commit message: Add files via upload
More routing of the PCB....  Slowly getting there.
Parts:
- moved TP501 402.4 mm to (3.45, 135.0)
- moved R515 368.3 mm to (24.4, 142.2)
- moved R516 368.3 mm to (24.4, 144.6)
- moved C527 365.1 mm to (15.8, 112.4)
- moved TP106 312.6 mm to (105.4, 112.3)
- moved TP502 305.8 mm to (101.8, 132.4)
- moved C528 281.8 mm to (102.8, 114.6)
- moved C504 225.0 mm to (6.25, 130.3)
- moved C524 224.0 mm to (10.5, 138.8)
- moved R508 224.0 mm to (16.1, 138.8)
- moved C506 224.0 mm to (7.67, 133.4)
- moved C507 224.0 mm to (23.4, 127.8)
- moved C509 224.0 mm to (7.67, 135.8)
- moved C511 224.0 mm to (7.67, 128.7)
- moved C513 224.0 mm to (13.3, 131.8)
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Routing:
- net (no net): track 256.8 -> 0.00 mm, vias 8 -> 0
- net /LINK2_AUD: track 72.7 -> 328.6 mm, vias 3 -> 6
- net /LINK1_AUD: track 72.4 -> 279.8 mm
- net /CH1/LOCAL_LINK: track 72.8 -> 225.2 mm
- net +12V: track 107.4 -> 258.6 mm, vias 0 -> 3
- net /PTT1D: track 0.00 -> 107.4 mm, vias 0 -> 3
- net /~CTCSS1: track 0.00 -> 101.2 mm, vias 0 -> 3
- net /COR1: track 0.00 -> 96.7 mm, vias 0 -> 3
- net /CH1/TONE_FROM_PI: track 19.2 -> 90.7 mm, vias 2 -> 4
- net MISO_5: track 110.2 -> 41.9 mm, vias 8 -> 2
- net /SDA0_33: track 0.00 -> 61.0 mm
- net +5V: track 272.9 -> 213.8 mm, vias 23 -> 9
- net /SCL0_33: track 0.00 -> 58.6 mm
- net /Spares, GPIO, and ADC/ADC0: track 8.98 -> 56.7 mm, vias 0 -> 1
- net /Spares, GPIO, and ADC/ADC_VIN: track 46.1 -> 1.55 mm, vias 2 -> 0
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