File: sch_pcb/soundcard.sch (KiCad schematic (older format))
At the start: 77 parts, among them J501 MicroUSB, Q501 BSR315PH6327XTSA1, U501 CM108B, U502 CM108B, U503 TUSB2036, U504 MCP1703A-3302/MB, U505 CM108B, Y501 6MHz

Commit message: BOM scrub
Parts:
- C501, C503, C505, C507, C513, C514, C515, C516, C517, C518, C519, C520, C533, C534, C535, C537, C538, C539: value 4u7 -> 4.7u
- C502, C504, C506, C508, C521, C522, C536, C543: value 100n -> 0.1u
- C509, C510, C511, C512, C527, C528, C540, C541, C542: footprint lib:smd0603 -> lib:smd0805
- R503, R504, R505, R506, R507, R508, R519, R520: value 22R -> 22
- R515, R516, R523: value 33R -> 33
Changed lines of the file:
@@
 P 7300 1225
 F 0 "C504" H 7350 1325 50  0000 L CNN
-F 1 "100n" H 7350 1125 50  0000 L CNN
+F 1 "0.1u" H 7350 1125 50  0000 L CNN
 F 2 "lib:smd0603" H 7338 1075 50  0001 C CNN
 F 3 "" H 7300 1225 50  0001 C CNN
@@
 P 6900 1225
 F 0 "C503" H 6975 1325 50  0000 L CNN
-F 1 "4u7" H 6975 1125 50  0000 L CNN
+F 1 "4.7u" H 6975 1125 50  0000 L CNN
 F 2 "lib:smd0603" H 6938 1075 50  0001 C CNN
 F 3 "" H 6900 1225 50  0001 C CNN
@@
 P 4600 1225
 F 0 "C508" H 4715 1271 50  0000 L CNN
-F 1 "100n" H 4715 1180 50  0000 L CNN
+F 1 "0.1u" H 4715 1180 50  0000 L CNN
 F 2 "lib:smd0603" H 4638 1075 50  0001 C CNN
 F 3 "" H 4600 1225 50  0001 C CNN
@@
 P 4150 1225
 F 0 "C507" H 4265 1271 50  0000 L CNN
-F 1 "4u7" H 4265 1180 50  0000 L CNN
+F 1 "4.7u" H 4265 1180 50  0000 L CNN
 F 2 "lib:smd0603" H 4188 1075 50  0001 C CNN
 F 3 "" H 4150 1225 50  0001 C CNN
@@
 P 6850 3500
 F 0 "C514" H 6965 3546 50  0000 L CNN
-F 1 "4u7" H 6965 3455 50  0000 L CNN
+F 1 "4.7u" H 6965 3455 50  0000 L CNN
 F 2 "lib:smd0603" H 6888 3350 50  0001 C CNN
 F 3 "" H 6850 3500 50  0001 C CNN
@@
 F 0 "C512" V 7025 2850 50  0000 C CNN
 F 1 "10u" V 7025 3175 50  0000 C CNN
-F 2 "lib:smd0603" H 7013 2900 50  0001 C CNN
+F 2 "lib:smd0805" H 7013 2900 50  0001 C CNN
 F 3 "" H 6975 3050 50  0001 C CNN
 	1    6975 3050
@@
 F 0 "C510" V 7025 2625 50  0000 C CNN
 F 1 "10u" V 7025 2925 50  0000 C CNN
-F 2 "lib:smd0603" H 7013 2650 50  0001 C CNN
+F 2 "lib:smd0805" H 7013 2650 50  0001 C CNN
 F 3 "" H 6975 2800 50  0001 C CNN
 	1    6975 2800
@@
 P 4600 3825
 F 0 "C520" H 4715 3871 50  0000 L CNN
-F 1 "4u7" H 4650 3725 50  0000 L CNN
+F 1 "4.7u" H 4650 3725 50  0000 L CNN
 F 2 "lib:smd0603" H 4638 3675 50  0001 C CNN
 F 3 "" H 4600 3825 50  0001 C CNN
@@
 P 4300 3825
 F 0 "C519" H 4350 3925 50  0000 L CNN
-F 1 "4u7" H 4350 3725 50  0000 L CNN
+F 1 "4.7u" H 4350 3725 50  0000 L CNN
 F 2 "lib:smd0603" H 4338 3675 50  0001 C CNN
 F 3 "" H 4300 3825 50  0001 C CNN
@@
 P 4025 3825
 F 0 "C518" H 4075 3925 50  0000 L CNN
-F 1 "4u7" H 4075 3725 50  0000 L CNN
+F 1 "4.7u" H 4075 3725 50  0000 L CNN
 F 2 "lib:smd0603" H 4063 3675 50  0001 C CNN
 F 3 "" H 4025 3825 50  0001 C CNN
@@
 P 3825 1225
 F 0 "C502" H 3850 1325 50  0000 L CNN
-F 1 "100n" H 3850 1125 50  0000 L CNN
+F 1 "0.1u" H 3850 1125 50  0000 L CNN
 F 2 "lib:smd0603" H 3863 1075 50  0001 C CNN
 F 3 "" H 3825 1225 50  0001 C CNN
@@
 P 3500 1225
 F 0 "C501" H 3550 1325 50  0000 L CNN
-F 1 "4u7" H 3550 1125 50  0000 L CNN
+F 1 "4.7u" H 3550 1125 50  0000 L CNN
 F 2 "lib:smd0603" H 3538 1075 50  0001 C CNN
 F 3 "" H 3500 1225 50  0001 C CNN
@@
 P 1325 1225
 F 0 "C506" H 1440 1271 50  0000 L CNN
-F 1 "100n" H 1440 1180 50  0000 L CNN
+F 1 "0.1u" H 1440 1180 50  0000 L CNN
 F 2 "lib:smd0603" H 1363 1075 50  0001 C CNN
 F 3 "" H 1325 1225 50  0001 C CNN
@@
 P 875 1225
 F 0 "C505" H 990 1271 50  0000 L CNN
-F 1 "4u7" H 990 1180 50  0000 L CNN
+F 1 "4.7u" H 990 1180 50  0000 L CNN
 F 2 "lib:smd0603" H 913 1075 50  0001 C CNN
 F 3 "" H 875 1225 50  0001 C CNN
@@
 P 3500 3500
 F 0 "C513" H 3615 3546 50  0000 L CNN
-F 1 "4u7" H 3615 3455 50  0000 L CNN
+F 1 "4.7u" H 3615 3455 50  0000 L CNN
 F 2 "lib:smd0603" H 3538 3350 50  0001 C CNN
 F 3 "" H 3500 3500 50  0001 C CNN
@@
 F 0 "C511" V 3675 2900 50  0000 C CNN
 F 1 "10u" V 3675 3175 50  0000 C CNN
-F 2 "lib:smd0603" H 3663 2900 50  0001 C CNN
+F 2 "lib:smd0805" H 3663 2900 50  0001 C CNN
 F 3 "" H 3625 3050 50  0001 C CNN
 	1    3625 3050
@@
 F 0 "C509" V 3675 2625 50  0000 C CNN
 F 1 "10u" V 3675 2925 50  0000 C CNN
-F 2 "lib:smd0603" H 3663 2650 50  0001 C CNN
+F 2 "lib:smd0805" H 3663 2650 50  0001 C CNN
 F 3 "" H 3625 2800 50  0001 C CNN
 	1    3625 2800
@@
 P 1250 3825
 F 0 "C517" H 1365 3871 50  0000 L CNN
-F 1 "4u7" H 1325 3725 50  0000 L CNN
+F 1 "4.7u" H 1325 3725 50  0000 L CNN
 F 2 "lib:smd0603" H 1288 3675 50  0001 C CNN
 F 3 "" H 1250 3825 50  0001 C CNN
@@
 P 950 3825
 F 0 "C516" H 1000 3925 50  0000 L CNN
-F 1 "4u7" H 1000 3725 50  0000 L CNN
+F 1 "4.7u" H 1000 3725 50  0000 L CNN
 F 2 "lib:smd0603" H 988 3675 50  0001 C CNN
 F 3 "" H 950 3825 50  0001 C CNN
@@
 P 675 3825
 F 0 "C515" H 725 3925 50  0000 L CNN
-F 1 "4u7" H 725 3725 50  0000 L CNN
+F 1 "4.7u" H 725 3725 50  0000 L CNN
 F 2 "lib:smd0603" H 713 3675 50  0001 C CNN
 F 3 "" H 675 3825 50  0001 C CNN
@@
 P 1775 5300
 F 0 "R504" V 1700 5300 50  0000 C CNN
-F 1 "22R" V 1775 5300 50  0000 C CNN
+F 1 "22" V 1775 5300 50  0000 C CNN
 F 2 "lib:smd0603" V 1705 5300 50  0001 C CNN
 F 3 "" H 1775 5300 50  0001 C CNN
@@
 P 1775 5400
 F 0 "R506" V 1850 5400 50  0000 C CNN
-F 1 "22R" V 1775 5400 50  0000 C CNN
+F 1 "22" V 1775 5400 50  0000 C CNN
 F 2 "lib:smd0603" V 1705 5400 50  0001 C CNN
 F 3 "" H 1775 5400 50  0001 C CNN
@@
 P 4025 4325
 F 0 "C521" V 3950 4175 50  0000 C CNN
-F 1 "100n" V 3950 4475 50  0000 C CNN
+F 1 "0.1u" V 3950 4475 50  0000 C CNN
 F 2 "lib:smd0603" H 4063 4175 50  0001 C CNN
 F 3 "" H 4025 4325 50  0001 C CNN
@@
 P 4850 5200
 F 0 "R503" V 4775 5200 50  0000 C CNN
-F 1 "22R" V 4850 5200 50  0000 C CNN
+F 1 "22" V 4850 5200 50  0000 C CNN
 F 2 "lib:smd0603" V 4780 5200 50  0001 C CNN
 F 3 "" H 4850 5200 50  0001 C CNN
@@
 P 5125 5300
 F 0 "R505" V 5200 5300 50  0000 C CNN
-F 1 "22R" V 5125 5300 50  0000 C CNN
+F 1 "22" V 5125 5300 50  0000 C CNN
 F 2 "lib:smd0603" V 5055 5300 50  0001 C CNN
 F 3 "" H 5125 5300 50  0001 C CNN
@@
 P 4850 5600
 F 0 "R507" V 4775 5600 50  0000 C CNN
-F 1 "22R" V 4850 5600 50  0000 C CNN
+F 1 "22" V 4850 5600 50  0000 C CNN
 F 2 "lib:smd0603" V 4780 5600 50  0001 C CNN
 F 3 "" H 4850 5600 50  0001 C CNN
@@
 P 5125 5700
 F 0 "R508" V 5200 5700 50  0000 C CNN
-F 1 "22R" V 5125 5700 50  0000 C CNN
+F 1 "22" V 5125 5700 50  0000 C CNN
 F 2 "lib:smd0603" V 5055 5700 50  0001 C CNN
 F 3 "" H 5125 5700 50  0001 C CNN
@@
 P 1925 4775
 F 0 "C522" H 1700 4875 50  0000 L CNN
-F 1 "100n" H 1700 4700 50  0000 L CNN
+F 1 "0.1u" H 1700 4700 50  0000 L CNN
 F 2 "lib:smd0603" H 1963 4625 50  0001 C CNN
 F 3 "" H 1925 4775 50  0001 C CNN
@@
 P 2450 1000
 F 0 "R515" V 2525 1000 50  0000 C CNN
-F 1 "33R" V 2450 1000 50  0000 C CNN
+F 1 "33" V 2450 1000 50  0000 C CNN
 F 2 "lib:smd0603" V 2380 1000 50  0001 C CNN
 F 3 "" H 2450 1000 50  0001 C CNN
@@
 P 5800 1000
 F 0 "R516" V 5875 1000 50  0000 C CNN
-F 1 "33R" V 5800 1000 50  0000 C CNN
+F 1 "33" V 5800 1000 50  0000 C CNN
 F 2 "lib:smd0603" V 5730 1000 50  0001 C CNN
 F 3 "" H 5800 1000 50  0001 C CNN
@@
 F 0 "C527" V 3675 2425 50  0000 C CNN
 F 1 "10u" V 3675 2725 50  0000 C CNN
-F 2 "lib:smd0603" H 3663 2450 50  0001 C CNN
+F 2 "lib:smd0805" H 3663 2450 50  0001 C CNN
 F 3 "" H 3625 2600 50  0001 C CNN
 	1    3625 2600
@@
 F 0 "C528" V 7025 2425 50  0000 C CNN
 F 1 "10u" V 7025 2725 50  0000 C CNN
-F 2 "lib:smd0603" H 7013 2450 50  0001 C CNN
+F 2 "lib:smd0805" H 7013 2450 50  0001 C CNN
 F 3 "" H 6975 2600 50  0001 C CNN
 	1    6975 2600
@@
 P 10650 1225
 F 0 "C543" H 10765 1271 50  0000 L CNN
-F 1 "100n" H 10765 1180 50  0000 L CNN
+F 1 "0.1u" H 10765 1180 50  0000 L CNN
 F 2 "lib:smd0603" H 10688 1075 50  0001 C CNN
 F 3 "" H 10650 1225 50  0001 C CNN
@@
 P 10300 1225
 F 0 "C539" H 10375 1350 50  0000 L CNN
-F 1 "4u7" H 10415 1180 50  0000 L CNN
+F 1 "4.7u" H 10415 1180 50  0000 L CNN
 F 2 "lib:smd0603" H 10338 1075 50  0001 C CNN
 F 3 "" H 10300 1225 50  0001 C CNN
@@
 P 8000 1225
 F 0 "C536" H 8115 1271 50  0000 L CNN
-F 1 "100n" H 8115 1180 50  0000 L CNN
+F 1 "0.1u" H 8115 1180 50  0000 L CNN
 F 2 "lib:smd0603" H 8038 1075 50  0001 C CNN
 F 3 "" H 8000 1225 50  0001 C CNN
@@
 P 7575 1225
 F 0 "C534" H 7690 1271 50  0000 L CNN
-F 1 "4u7" H 7690 1180 50  0000 L CNN
+F 1 "4.7u" H 7690 1180 50  0000 L CNN
 F 2 "lib:smd0603" H 7613 1075 50  0001 C CNN
 F 3 "" H 7575 1225 50  0001 C CNN
@@
 P 10250 3500
 F 0 "C538" H 10365 3546 50  0000 L CNN
-F 1 "4u7" H 10365 3455 50  0000 L CNN
+F 1 "4.7u" H 10365 3455 50  0000 L CNN
 F 2 "lib:smd0603" H 10288 3350 50  0001 C CNN
 F 3 "" H 10250 3500 50  0001 C CNN
@@
 F 0 "C542" V 10425 2850 50  0000 C CNN
 F 1 "10u" V 10425 3175 50  0000 C CNN
-F 2 "lib:smd0603" H 10413 2900 50  0001 C CNN
+F 2 "lib:smd0805" H 10413 2900 50  0001 C CNN
 F 3 "" H 10375 3050 50  0001 C CNN
 	1    10375 3050
@@
 F 0 "C541" V 10425 2625 50  0000 C CNN
 F 1 "10u" V 10425 2925 50  0000 C CNN
-F 2 "lib:smd0603" H 10413 2650 50  0001 C CNN
+F 2 "lib:smd0805" H 10413 2650 50  0001 C CNN
 F 3 "" H 10375 2800 50  0001 C CNN
 	1    10375 2800
@@
 P 8000 3825
 F 0 "C537" H 8115 3871 50  0000 L CNN
-F 1 "4u7" H 8050 3725 50  0000 L CNN
+F 1 "4.7u" H 8050 3725 50  0000 L CNN
 F 2 "lib:smd0603" H 8038 3675 50  0001 C CNN
 F 3 "" H 8000 3825 50  0001 C CNN
@@
 P 7700 3825
 F 0 "C535" H 7750 3925 50  0000 L CNN
-F 1 "4u7" H 7750 3725 50  0000 L CNN
+F 1 "4.7u" H 7750 3725 50  0000 L CNN
 F 2 "lib:smd0603" H 7738 3675 50  0001 C CNN
 F 3 "" H 7700 3825 50  0001 C CNN
@@
 P 7425 3825
 F 0 "C533" H 7475 3925 50  0000 L CNN
-F 1 "4u7" H 7475 3725 50  0000 L CNN
+F 1 "4.7u" H 7475 3725 50  0000 L CNN
 F 2 "lib:smd0603" H 7463 3675 50  0001 C CNN
 F 3 "" H 7425 3825 50  0001 C CNN
@@
 P 9200 1000
 F 0 "R523" V 9275 1000 50  0000 C CNN
-F 1 "33R" V 9200 1000 50  0000 C CNN
+F 1 "33" V 9200 1000 50  0000 C CNN
 F 2 "lib:smd0603" V 9130 1000 50  0001 C CNN
 F 3 "" H 9200 1000 50  0001 C CNN
@@
 F 0 "C540" V 10425 2425 50  0000 C CNN
 F 1 "10u" V 10425 2725 50  0000 C CNN
-F 2 "lib:smd0603" H 10413 2450 50  0001 C CNN
+F 2 "lib:smd0805" H 10413 2450 50  0001 C CNN
 F 3 "" H 10375 2600 50  0001 C CNN
 	1    10375 2600
@@
 P 4850 6000
 F 0 "R519" V 4775 6000 50  0000 C CNN
-F 1 "22R" V 4850 6000 50  0000 C CNN
+F 1 "22" V 4850 6000 50  0000 C CNN
 F 2 "lib:smd0603" V 4780 6000 50  0001 C CNN
 F 3 "" H 4850 6000 50  0001 C CNN
@@
 P 5125 6100
 F 0 "R520" V 5200 6100 50  0000 C CNN
-F 1 "22R" V 5125 6100 50  0000 C CNN
+F 1 "22" V 5125 6100 50  0000 C CNN
 F 2 "lib:smd0603" V 5055 6100 50  0001 C CNN
 F 3 "" H 5125 6100 50  0001 C CNN
